File: hardware/bedlight-nucleo/bedlight-nucleo.sch (KiCad schematic (older format))
At the start: 10 parts, among them SW1 SW_Push, SW2 SW_Push, SW3 SW_Push, SW4 SW_Push, U1 Nucleo-32, U2 ULN2003A

Commit message: Footprints partially placed
Parts:
- U1: footprint Module:Arduino_Nano -> bedlight-nucleo:Nucleo-32
Connections:
- net labels added: OUT1, OUT2, OUT3, OUT4
- wire segments 44 -> 52
Changed lines of the file:
@@
 $EndDescr
 Wire Wire Line
-	4300 4300 3650 4300
-Wire Wire Line
 	4300 4200 3650 4200
 Wire Wire Line
 	4300 4100 3650 4100
+Wire Wire Line
+	4300 4000 3650 4000
 Wire Wire Line
 	5000 2600 5000 2150
@@
 F 0 "U1" H 5400 4600 50  0000 C CNN
 F 1 "Nucleo-32" H 5550 4750 50  0000 C CNN
-F 2 "Module:Arduino_Nano" H 4800 3600 50  0001 C CIN
+F 2 "bedlight-nucleo:Nucleo-32" H 4800 3600 50  0001 C CIN
 F 3 "https://www.arduino.cc/en/uploads/Main/ArduinoNanoManual23.pdf" H 4800 3600 50  0001 C CNN
 	1    4800 3600
@@
 Text Label 3750 5750 0    50   ~ 0
 LED_RED
-Text Label 3750 4300 0    50   ~ 0
+Text Label 3750 4200 0    50   ~ 0
 LED_BLUE
-Text Label 3750 4200 0    50   ~ 0
+Text Label 3750 4100 0    50   ~ 0
 LED_GREEN
-Text Label 3750 4100 0    50   ~ 0
+Text Label 3750 4000 0    50   ~ 0
 LED_RED
 $Comp
@@
 	1    0    0    -1
 $EndComp
+Wire Wire Line
+	3650 5850 4350 5850
+Wire Wire Line
+	4350 5950 3650 5950
+Wire Wire Line
+	4350 6050 3650 6050
+Wire Wire Line
+	4350 6150 3650 6150
+Text Label 3750 5850 0    50   ~ 0
+OUT1
+Text Label 3750 5950 0    50   ~ 0
+OUT2
+Text Label 3750 6050 0    50   ~ 0
+OUT3
+Text Label 3750 6150 0    50   ~ 0
+OUT4
+Wire Wire Line
+	4300 3900 3650 3900
+Wire Wire Line
+	4300 3800 3650 3800
+Wire Wire Line
+	4300 3700 3650 3700
+Text Label 3750 3900 0    50   ~ 0
+OUT1
+Text Label 3750 3800 0    50   ~ 0
+OUT2
+Text Label 3750 3700 0    50   ~ 0
+OUT3
+Wire Wire Line
+	4300 3600 3650 3600
+Text Label 3750 3600 0    50   ~ 0
+OUT4
 $EndSCHEMATC

Commit message: Added mounting holes
Parts:
- added H1, H2, H3, H4, H5, H6, H7, H8: MountingHole, MountingHole:MountingHole_3.2mm_M3_DIN965_Pad, symbol Mechanical:MountingHole
Changed lines of the file:
@@
 Text Label 3750 3600 0    50   ~ 0
 OUT4
+$Comp
+L Mechanical:MountingHole H1
+U 1 1 5F14D77B
+P 9900 2450
+F 0 "H1" H 10000 2496 50  0000 L CNN
+F 1 "MountingHole" H 10000 2405 50  0000 L CNN
+F 2 "MountingHole:MountingHole_3.2mm_M3_DIN965_Pad" H 9900 2450 50  0001 C CNN
+F 3 "~" H 9900 2450 50  0001 C CNN
+	1    9900 2450
+	1    0    0    -1
+$EndComp
+$Comp
+L Mechanical:MountingHole H2
+U 1 1 5F14DF65
+P 9900 2650
+F 0 "H2" H 10000 2696 50  0000 L CNN
+F 1 "MountingHole" H 10000 2605 50  0000 L CNN
+F 2 "MountingHole:MountingHole_3.2mm_M3_DIN965_Pad" H 9900 2650 50  0001 C CNN
+F 3 "~" H 9900 2650 50  0001 C CNN
+	1    9900 2650
+	1    0    0    -1
+$EndComp
+$Comp
+L Mechanical:MountingHole H3
+U 1 1 5F14E2E9
+P 9900 2850
+F 0 "H3" H 10000 2896 50  0000 L CNN
+F 1 "MountingHole" H 10000 2805 50  0000 L CNN
+F 2 "MountingHole:MountingHole_3.2mm_M3_DIN965_Pad" H 9900 2850 50  0001 C CNN
+F 3 "~" H 9900 2850 50  0001 C CNN
+	1    9900 2850
+	1    0    0    -1
+$EndComp
+$Comp
+L Mechanical:MountingHole H4
+U 1 1 5F14E57D
+P 9900 3050
+F 0 "H4" H 10000 3096 50  0000 L CNN
+F 1 "MountingHole" H 10000 3005 50  0000 L CNN
+F 2 "MountingHole:MountingHole_3.2mm_M3_DIN965_Pad" H 9900 3050 50  0001 C CNN
+F 3 "~" H 9900 3050 50  0001 C CNN
+	1    9900 3050
+	1    0    0    -1
+$EndComp
+$Comp
+L Mechanical:MountingHole H5
+U 1 1 5F1504EC
+P 9900 3250
+F 0 "H5" H 10000 3296 50  0000 L CNN
+F 1 "MountingHole" H 10000 3205 50  0000 L CNN
+F 2 "MountingHole:MountingHole_3.2mm_M3_DIN965_Pad" H 9900 3250 50  0001 C CNN
+F 3 "~" H 9900 3250 50  0001 C CNN
+	1    9900 3250
+	1    0    0    -1
+$EndComp
+$Comp
+L Mechanical:MountingHole H6
+U 1 1 5F1507A3
+P 9900 3450
+F 0 "H6" H 10000 3496 50  0000 L CNN
+F 1 "MountingHole" H 10000 3405 50  0000 L CNN
+F 2 "MountingHole:MountingHole_3.2mm_M3_DIN965_Pad" H 9900 3450 50  0001 C CNN
+F 3 "~" H 9900 3450 50  0001 C CNN
+	1    9900 3450
+	1    0    0    -1
+$EndComp
+$Comp
+L Mechanical:MountingHole H7
+U 1 1 5F1509F3
+P 9900 3650
+F 0 "H7" H 10000 3696 50  0000 L CNN
+F 1 "MountingHole" H 10000 3605 50  0000 L CNN
+F 2 "MountingHole:MountingHole_3.2mm_M3_DIN965_Pad" H 9900 3650 50  0001 C CNN
+F 3 "~" H 9900 3650 50  0001 C CNN
+	1    9900 3650
+	1    0    0    -1
+$EndComp
+$Comp
+L Mechanical:MountingHole H8
+U 1 1 5F150BCE
+P 9900 3850
+F 0 "H8" H 10000 3896 50  0000 L CNN
+F 1 "MountingHole" H 10000 3805 50  0000 L CNN
+F 2 "MountingHole:MountingHole_3.2mm_M3_DIN965_Pad" H 9900 3850 50  0001 C CNN
+F 3 "~" H 9900 3850 50  0001 C CNN
+	1    9900 3850
+	1    0    0    -1
+$EndComp
 $EndSCHEMATC

Commit message: Resistor value set to 47R
Parts:
- R1, R2, R3: value R -> 47R
Changed lines of the file:
@@
 P 5550 5550
 F 0 "R1" V 5500 5300 50  0000 C CNN
-F 1 "R" V 5500 5750 50  0000 C CNN
+F 1 "47R" V 5500 5750 50  0000 C CNN
 F 2 "Resistor_THT:R_Axial_DIN0207_L6.3mm_D2.5mm_P10.16mm_Horizontal" V 5480 5550 50  0001 C CNN
 F 3 "~" H 5550 5550 50  0001 C CNN
@@
 P 5550 5650
 F 0 "R2" V 5500 5400 50  0000 C CNN
-F 1 "R" V 5500 5850 50  0000 C CNN
+F 1 "47R" V 5500 5850 50  0000 C CNN
 F 2 "Resistor_THT:R_Axial_DIN0207_L6.3mm_D2.5mm_P10.16mm_Horizontal" V 5480 5650 50  0001 C CNN
 F 3 "~" H 5550 5650 50  0001 C CNN
@@
 P 5550 5750
 F 0 "R3" V 5500 5500 50  0000 C CNN
-F 1 "R" V 5500 5950 50  0000 C CNN
+F 1 "47R" V 5500 5950 50  0000 C CNN
 F 2 "Resistor_THT:R_Axial_DIN0207_L6.3mm_D2.5mm_P10.16mm_Horizontal" V 5480 5750 50  0001 C CNN
 F 3 "~" H 5550 5750 50  0001 C CNN
